File: CAN_Power_Velleman/CAN_Power.kicad_pcb (KiCad board)
At the start: 2 copper layers, 19 parts, among them K1 CONN_3, P1 CONN_1, P2 CONN_1, P3 CONN_1, P4 CONN_2, P5 CONN_4, P6 CONN_1, P7 CONN_1, P8 CONN_1, P9 FUSE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

Commit message: Last update of modules before ordering PCBs
Parts:
- removed P4: CONN_2, bornier2
- added K2: CONN_3, bornier3, F.Cu at (112.0, 86.5)
- moved 1PIN 1.00 mm to (88.0, 263.0)
- moved 1PIN 1.00 mm to (136.0, 263.0)
Connections:
- U1 pad 17: GND -> GNDPWR
- U1 pad 18: GND -> GNDPWR
Routing:
- net GNDPWR: track 0.00 -> 268.6 mm, vias 0 -> 2
- net N-0000013: track 21.7 -> 16.4 mm
- net N-000004: track 21.7 -> 20.6 mm
