File: CAN_Power_Velleman/CAN_Power.sch (KiCad schematic (older format))
At the start: 11 parts, among them K1 CONN_3, P1 CONN_1, P2 CONN_1, P3 CONN_1, P4 CONN_2, P5 CONN_4, P6 CONN_1, P7 CONN_1, P8 CONN_1, P9 FUSE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

Commit message: Last update of modules before ordering PCBs
Parts:
- removed P4: CONN_2, symbol CONN_2
- added K2: CONN_3, symbol CONN_3
Connections:
- net GND: no longer U1.17 (Shield), U1.18 (Shield)
- net at P1.1: now also K2.2 (PM)
- net at P7.1: now also K2.3 (P3)
- new net GNDPWR: K2.1 (P1), U1.17 (Shield), U1.18 (Shield)
Changed lines of the file:
@@
 Sheet 1 1
 Title ""
-Date "26 oct 2014"
+Date "28 oct 2014"
 Rev ""
 Comp ""
@@
 Comment4 ""
 $EndDescr
-$Comp
-L CONN_2 P4
-U 1 1 544C2F30
-P 5450 2150
-F 0 "P4" V 5400 2150 40  0000 C CNN
-F 1 "CONN_2" V 5500 2150 40  0000 C CNN
-F 2 "" H 5450 2150 60  0000 C CNN
-F 3 "" H 5450 2150 60  0000 C CNN
-	1    5450 2150
-	0    -1   -1   0
-$EndComp
 $Comp
 L CONN_1 P1
@@
 $EndComp
 Wire Wire Line
-	5350 2500 5350 2850
-Wire Wire Line
-	5350 2850 5000 2850
+	5000 2850 5450 2850
 Wire Wire Line
 	5550 2500 5550 2850
@@
 	5900 5900 5900 6050
 Wire Wire Line
-	6500 5850 6500 7050
-Wire Wire Line
 	6500 5850 6200 5850
 Connection ~ 6200 5850
 Wire Wire Line
-	4350 6400 4350 7050
+	4350 2500 4350 7050
 Wire Wire Line
 	4350 7050 6500 7050
 Connection ~ 6500 6400
 Wire Wire Line
-	4400 6400 4350 6400
+	4000 6400 4400 6400
 $Comp
 L GND #PWR01
 U 1 1 544D5E6E
-P 6850 6650
-F 0 "#PWR01" H 6850 6650 30  0001 C CNN
-F 1 "GND" H 6850 6580 30  0001 C CNN
-F 2 "" H 6850 6650 60  0000 C CNN
-F 3 "" H 6850 6650 60  0000 C CNN
-	1    6850 6650
-	1    0    0    -1
-$EndComp
-Wire Wire Line
-	6500 6550 6850 6550
-Wire Wire Line
-	6850 6550 6850 6650
-Connection ~ 6500 6550
+P 6500 6100
+F 0 "#PWR01" H 6500 6100 30  0001 C CNN
+F 1 "GND" H 6500 6030 30  0001 C CNN
+F 2 "" H 6500 6100 60  0000 C CNN
+F 3 "" H 6500 6100 60  0000 C CNN
+	1    6500 6100
+	1    0    0    -1
+$EndComp
 NoConn ~ 5350 5250
 $Comp
@@
 Wire Wire Line
 	5750 5550 5750 5500
+Wire Wire Line
+	6500 5850 6500 6100
+Wire Wire Line
+	6500 7050 6500 6400
+$Comp
+L GNDPWR #PWR02
+U 1 1 544FF692
+P 4000 6650
+F 0 "#PWR02" H 4000 6700 40  0001 C CNN
+F 1 "GNDPWR" H 4000 6570 40  0000 C CNN
+F 2 "" H 4000 6650 60  0000 C CNN
+F 3 "" H 4000 6650 60  0000 C CNN
+	1    4000 6650
+	1    0    0    -1
+$EndComp
+Wire Wire Line
+	4000 6650 4000 6400
+Connection ~ 4350 6400
+$Comp
+L CONN_3 K2
+U 1 1 544FF6DC
+P 5450 2150
+F 0 "K2" V 5400 2150 50  0000 C CNN
+F 1 "CONN_3" V 5500 2150 40  0000 C CNN
+F 2 "" H 5450 2150 60  0000 C CNN
+F 3 "" H 5450 2150 60  0000 C CNN
+	1    5450 2150
+	0    -1   -1   0
+$EndComp
+Wire Wire Line
+	5450 2850 5450 2500
+Wire Wire Line
+	5350 2500 4350 2500
 $EndSCHEMATC
