File: USB2CAN_SUBD9_RJ45/vscp_usb2can.kicad_pcb (KiCad board)
At the start: 2 copper layers, 6 parts, among them P1 Sub-D 9, U1 RJ45_DUAL

Commit message: Last update of modules before ordering PCBs
Parts:
- removed P1: Sub-D 9, PIN_ARRAY_4x1
- added K1: CONN_3, PIN_ARRAY_3X1, F.Cu at (185.6, 150.5)
- moved 1PIN 1.00 mm to (204.0, 178.0)
- moved 1PIN 1.00 mm to (167.0, 178.0)
Connections:
- U1 pad 17: N-000005 (its old number) -> (no net)
- U1 pad 18: N-000005 (its old number) -> (no net)
Routing:
- net N-000005 (its old number): track 62.7 -> 0.00 mm
