File: USB2CAN_SUBD9_RJ45/vscp_usb2can.sch (KiCad schematic (older format))
At the start: 2 parts, among them P1 Sub-D 9, U1 RJ45_DUAL

Commit message: Last update of modules before ordering PCBs
Parts:
- removed P1: Sub-D 9, symbol CONN_4
- added K1: CONN_3, symbol CONN_3
Connections:
- net GND: now also K1.1 (P1)
- net at U1.12, U1.4: now also K1.2 (PM)
- net at U1.13, U1.5: now also K1.3 (P3)
- net at U1.17 (Shield): no longer U1.18 (Shield)
- no-connect marks 0 -> 2
Changed lines of the file:
@@
 Sheet 1 1
 Title ""
-Date "27 oct 2014"
+Date "28 oct 2014"
 Rev ""
 Comp ""
@@
 Wire Wire Line
 	5000 3500 5000 4350
-Wire Wire Line
-	4400 3350 4400 5300
 Connection ~ 5400 3850
-Wire Wire Line
-	6500 4700 6500 5300
-Wire Wire Line
-	6500 5300 4400 5300
-Connection ~ 4400 4700
 Wire Wire Line
 	6200 3950 6200 4350
@@
 Connection ~ 5600 3150
 $Comp
-L CONN_4 P1
-U 1 1 544EA50F
-P 5450 2450
-F 0 "P1" V 5400 2450 50  0000 C CNN
-F 1 "Sub-D 9" V 5500 2450 50  0000 C CNN
-F 2 "" H 5450 2450 60  0000 C CNN
-F 3 "" H 5450 2450 60  0000 C CNN
-	1    5450 2450
-	0    -1   -1   0
-$EndComp
-$Comp
 L GND #PWR01
 U 1 1 544D715A
@@
 Wire Wire Line
 	6450 3850 5400 3850
-Wire Wire Line
-	5300 2800 5300 3350
-Wire Wire Line
-	5300 3350 4400 3350
+NoConn ~ 4400 4700
+NoConn ~ 6500 4700
+$Comp
+L CONN_3 K1
+U 1 1 544FFEF3
+P 5500 2450
+F 0 "K1" V 5450 2450 50  0000 C CNN
+F 1 "CONN_3" V 5550 2450 40  0000 C CNN
+F 2 "" H 5500 2450 60  0000 C CNN
+F 3 "" H 5500 2450 60  0000 C CNN
+	1    5500 2450
+	0    -1   -1   0
+$EndComp
 $EndSCHEMATC
